File: KiCAD/ardHydroponic/ardHydroponic.kicad_pcb (KiCad board)
At the start: 2 copper layers, 7 parts, among them J1 3-pin_IRF5320_MOSFET_module_h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, J2 3-pin_IRF5320_MOSFET_module_h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, J3 3-pin_IRF5320_MOSFET_module_h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, J4 3-pin_IRF5320_MOSFET_module_h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, J5 4-pin_I2C_LCD_header, U1 DS18B20

Commit message: new pins, schematics
Parts:
- removed J4: 3-pin_IRF5320_MOSFET_module_header, My_Headers:3-pin_IRF5320_MOSFET_module_header_large
- removed J5: 4-pin_I2C_LCD_header, My_Headers:4-pin_I2C_LCD_header_larger
- added R1: 4.7k, My_Misc:R_Axial_DIN0207_L6.3mm_D2.5mm_P10.16mm_Horizontal_larger_pads, F.Cu at (134.6, 99.1)
- added R2: 10k, My_Misc:R_Axial_DIN0207_L6.3mm_D2.5mm_P10.16mm_Horizontal_larger_pads, F.Cu at (160.7, 94.0)
- added R3: 10k, My_Misc:R_Axial_DIN0207_L6.3mm_D2.5mm_P10.16mm_Horizontal_larger_pads, F.Cu at (160.7, 98.4)
- added R4: 10k, My_Misc:R_Axial_DIN0207_L6.3mm_D2.5mm_P10.16mm_Horizontal_larger_pads, F.Cu at (160.7, 102.9)
- added R5: 10k, My_Misc:R_Axial_DIN0207_L6.3mm_D2.5mm_P10.16mm_Horizontal_larger_pads, F.Cu at (160.7, 107.3)
- added R6: 10k, My_Misc:R_Axial_DIN0207_L6.3mm_D2.5mm_P10.16mm_Horizontal_larger_pads, F.Cu at (160.7, 111.8)
- added U2: pH sensor, My_Headers:3-pin_DFRobot_Gravity_pH-sensor_header_large, F.Cu at (120.0, 101.6)
- added U3: TDS meter, My_Headers:3-pin_DFRobot_Gravity_TDS-meter_header_large, F.Cu at (128.3, 101.6)
- added U4: Power in, My_Parts:2-pole_power_in_screw_terminal, F.Cu at (105.4, 102.9)
- J1: value 3-pin_IRF5320_MOSFET_module_header -> LCD display; footprint My_Headers:3-pin_IRF5320_MOSFET_module_header_large -> My_Headers:4-pin_I2C_LCD_header_larger
- J2: value 3-pin_IRF5320_MOSFET_module_header -> Buttons; footprint My_Headers:3-pin_IRF5320_MOSFET_module_header_large -> My_Parts:6-pole_5-NO_switch_screw_terminal
- J3: value 3-pin_IRF5320_MOSFET_module_header -> MOSFETs; footprint My_Headers:3-pin_IRF5320_MOSFET_module_header_large -> My_Parts:7-pole_6-MOSFET_screw_terminal
- U1: footprint My_Headers:3_pin_Dallas_1-wire_header_larger_pads -> My_Parts:3-pole_DS18B20_screw_terminal
- XA1: footprint My_Arduino:Arduino_Mega2560_Shield_large -> My_Arduino:Arduino_Mega2560_Shield__no_ICSP_large
- moved J2 45.7 mm to (179.7, 84.9)
- moved J1 39.4 mm to (163.2, 83.8), turned to 90 degrees
- moved U1 13.5 mm to (142.2, 109.9), turned to 90 degrees
- moved J3 9.44 mm to (153.0, 87.6), turned to 270 degrees
- moved XA1 1.27 mm to (100.3, 124.5)
Connections:
- J1 pad 1: Net-(J1-Pad1) -> +5V
- J1 pad 3: Net-(J1-Pad3) -> GND
- J2 pad 1: Net-(J2-Pad1) -> +5V
- J2 pad 2: Net-(J2-Pad2) -> button1
- J2 pad 3: Net-(J2-Pad3) -> button2
- J3 pad 1: Net-(J3-Pad1) -> +5V
- J3 pad 2: Net-(J3-Pad2) -> GND
- J3 pad 3: Net-(J3-Pad3) -> pH+
- U1 pad 1: Net-(U1-Pad1) -> GND
- U1 pad 2: Net-(U1-Pad2) -> dallas
- U1 pad 3: Net-(U1-Pad3) -> +5V
- XA1 pad 1: Net-(XA1-Pad1) -> nutrA
- XA1 pad 10: Net-(XA1-Pad10) -> +5V
- XA1 pad 100: Net-(XA1-Pad100) -> +6V
- XA1 pad 15: Net-(XA1-Pad15) -> stirrer
- XA1 pad 43: Net-(XA1-Pad43) -> Net-(J1-Pad7)
- XA1 pad 44: Net-(XA1-Pad44) -> Net-(J1-Pad5)
- XA1 pad 5: Net-(XA1-Pad5) -> nutrB
- XA1 pad 58: Net-(XA1-Pad58) -> dallas
- XA1 pad 6: Net-(XA1-Pad6) -> pH+
- XA1 pad 60: Net-(XA1-Pad60) -> button5
- XA1 pad 62: Net-(XA1-Pad62) -> GND
- XA1 pad 7: Net-(XA1-Pad7) -> pH-
- XA1 pad 72: Net-(XA1-Pad72) -> button4
- XA1 pad 74: Net-(XA1-Pad74) -> button3
- XA1 pad 76: Net-(XA1-Pad76) -> button2
- XA1 pad 78: Net-(XA1-Pad78) -> button1
Routing:
- net +5V: track 0.00 -> 284.9 mm, vias 0 -> 6
- net GND: track 0.00 -> 190.5 mm, vias 0 -> 2
- net dallas: track 0.00 -> 78.7 mm
- net +6V: track 0.00 -> 49.7 mm
- net button5: track 0.00 -> 39.9 mm
- net button4: track 0.00 -> 37.6 mm
- net Net-(U2-Pad3): track 0.00 -> 37.4 mm
- net button3: track 0.00 -> 35.4 mm
- net button2: track 0.00 -> 33.1 mm
- net Net-(U3-Pad3): track 0.00 -> 32.9 mm
- net stirrer: track 0.00 -> 32.5 mm
- net button1: track 0.00 -> 31.6 mm
- net nutrB: track 0.00 -> 29.7 mm
- net nutrA: track 0.00 -> 27.9 mm
- net pH-: track 0.00 -> 25.4 mm
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- added copper zone on B.Cu, net (none)
- added copper zone on B.Cu, net GND
Other:
- board outline added: 102.9 x 54.6 mm
- net class Default: clearance 0.2 -> 0.762; trace_width 0.25 -> 0.762; via_dia 0.8 -> 2.032
- rule trace_clearance: 0.2 -> 0.762
- board text added: "5V"
- board text added: "ardHydroponic Design: Jon Sagebrand github.com/jonsag"

Commit message: PCB
Routing:
- added copper zone on F.Cu, net (none)
- added copper zone on F.Cu, net GND
Other:
- board text added: "Power in"

Commit message: new schematics
Parts:
- moved R6 44.5 mm to (116.2, 109.2), turned to 90 degrees
- moved R5 40.1 mm to (120.7, 109.2), turned to 90 degrees
- moved J2 38.7 mm to (141.0, 85.1), turned to 270 degrees
- moved R4 36.1 mm to (125.1, 109.2), turned to 90 degrees
- moved R3 32.9 mm to (129.5, 109.2), turned to 90 degrees
- moved R2 30.7 mm to (134.0, 109.2), turned to 90 degrees
- moved J3 27.6 mm to (180.3, 83.8), turned to 0 degrees
- moved U1 22.3 mm to (164.5, 108.6), turned to 270 degrees
- moved U2 21.0 mm to (141.0, 102.2)
- moved U3 21.0 mm to (149.2, 102.2)
- moved R1 19.9 mm to (154.3, 95.9), turned to 180 degrees
- moved J1 2.84 mm to (164.5, 81.3)
- moved U4 2.54 mm to (108.0, 102.9)
Connections:
- R1 pad 1: +5V -> Net-(R1-Pad1)
- R1 pad 2: dallas -> +5V
- U1 pad 2: dallas -> Net-(R1-Pad1)
- XA1 pad 16: Net-(XA1-Pad16) -> button1
- XA1 pad 17: Net-(XA1-Pad17) -> button2
- XA1 pad 18: Net-(XA1-Pad18) -> button3
- XA1 pad 23: Net-(XA1-Pad23) -> button4
- XA1 pad 24: Net-(XA1-Pad24) -> button5
- XA1 pad 58: dallas -> Net-(XA1-Pad58)
- XA1 pad 60: button5 -> Net-(XA1-Pad60)
- XA1 pad 72: button4 -> Net-(XA1-Pad72)
- XA1 pad 74: button3 -> Net-(XA1-Pad74)
- XA1 pad 76: button2 -> Net-(XA1-Pad76)
- XA1 pad 78: button1 -> Net-(XA1-Pad78)
- XA1 pad 95: Net-(XA1-Pad95) -> Net-(R1-Pad1)
Routing:
- net dallas: track 78.7 -> 0.00 mm
- net GND: track 190.5 -> 238.2 mm
- net Net-(R1-Pad1): track 0.00 -> 29.5 mm
- net stirrer: track 32.5 -> 54.3 mm
- net nutrB: track 29.7 -> 50.1 mm
- net Net-(U2-Pad3): track 37.4 -> 18.8 mm
- net nutrA: track 27.9 -> 46.3 mm
- net Net-(U3-Pad3): track 32.9 -> 16.4 mm
- net pH-: track 25.4 -> 40.6 mm
- net pH+: track 22.9 -> 36.8 mm
- net +6V: track 49.7 -> 54.7 mm
- net Net-(J1-Pad7): track 21.3 -> 19.0 mm
- net Net-(J1-Pad5): track 21.7 -> 19.3 mm
- net button3: track 35.4 -> 33.1 mm
- net button2: track 33.1 -> 31.1 mm
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Other:
- board text added: "G"
- board text removed: "Power in"

Commit message: new PCB
Parts:
- moved R1 27.5 mm to (172.1, 116.8), turned to 0 degrees
- moved J1 14.9 mm to (179.1, 84.5)
- moved J3 13.3 mm to (180.3, 97.2), turned to 270 degrees
- moved U3 11.1 mm to (158.8, 108.0)
- moved U2 10.0 mm to (149.2, 108.0)
- moved R2 7.62 mm to (141.6, 109.2)
- moved R3 5.72 mm to (135.3, 109.2)
- moved U1 3.86 mm to (168.3, 108.0), turned to 90 degrees
- moved R4 3.81 mm to (128.9, 109.2)
- moved U4 3.42 mm to (104.8, 101.6), turned to 90 degrees
- moved R5 1.91 mm to (122.6, 109.2)
Routing:
- net GND: track 238.2 -> 67.6 mm, vias 2 -> 0
- net +5V: track 284.5 -> 197.2 mm, vias 6 -> 0
- net stirrer: track 54.3 -> 24.3 mm
- net nutrB: track 50.1 -> 25.1 mm
- net nutrA: track 46.3 -> 26.7 mm
- net pH-: track 40.6 -> 27.4 mm
- net Net-(U2-Pad3): track 18.8 -> 9.42 mm
- net pH+: track 36.8 -> 28.2 mm
- net Net-(J1-Pad5): track 19.3 -> 10.8 mm
- net Net-(J1-Pad7): track 19.0 -> 10.8 mm
- net Net-(U3-Pad3): track 16.4 -> 11.0 mm
- net +6V: track 54.7 -> 50.1 mm
- net button1: track 30.4 -> 31.9 mm
- net button2: track 31.1 -> 32.1 mm
- net button3: track 33.1 -> 34.0 mm
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Other:
- board text removed: "5V"
- board text removed: "G"

Commit message: kicad, programmer board
Parts:
- removed J1: LCD display, My_Headers:4-pin_I2C_LCD_header_larger
- removed J2: Buttons, My_Parts:6-pole_5-NO_switch_screw_terminal
- removed J3: MOSFETs, My_Parts:7-pole_6-MOSFET_screw_terminal
- removed R1: 4.7k, My_Misc:R_Axial_DIN0207_L6.3mm_D2.5mm_P10.16mm_Horizontal_larger_pads
- removed R2, R3, R4, R5, R6: 10k, My_Misc:R_Axial_DIN0207_L6.3mm_D2.5mm_P10.16mm_Horizontal_larger_pads
- removed U1: DS18B20, My_Parts:3-pole_DS18B20_screw_terminal
- removed U2: pH sensor, My_Headers:3-pin_DFRobot_Gravity_pH-sensor_header_large
- removed U3: TDS meter, My_Headers:3-pin_DFRobot_Gravity_TDS-meter_header_large
- removed U4: Power in, My_Parts:2-pole_power_in_screw_terminal
- added R7: 1k, My_Misc:R_Axial_DIN0207_L6.3mm_D2.5mm_P10.16mm_Horizontal_larger_pads, F.Cu at (126.4, 88.3)
- added R8: 2.2k, My_Misc:R_Axial_DIN0207_L6.3mm_D2.5mm_P10.16mm_Horizontal_larger_pads, F.Cu at (126.4, 97.2)
- added U10: ESP-01, My_Arduino:ESP-01_large, F.Cu at (143.5, 106.7)
- XA1: footprint My_Arduino:Arduino_Mega2560_Shield__no_ICSP_large -> My_Arduino:Arduino_Mega2560_Shield__no_ICSP_no_mount-holes_large
Connections:
- XA1 pad 25: Net-(XA1-Pad25) -> softRx
- XA1 pad 26: Net-(XA1-Pad26) -> softTx
- XA1 pad 3V3: Net-(XA1-Pad3V3) -> +3V3
- XA1 pad 64: Net-(XA1-Pad64) -> espReset
Routing:
- net +5V: track 197.2 -> 0.00 mm
- net espReset: track 0.00 -> 60.7 mm
- net softRx: track 0.00 -> 51.2 mm
- net +6V: track 50.1 -> 0.00 mm
- net +3V3: track 0.00 -> 44.6 mm, vias 0 -> 2
- net button5: track 38.0 -> 0.00 mm
- net button4: track 36.4 -> 0.00 mm
- net Net-(R7-Pad2): track 0.00 -> 35.1 mm
- net button3: track 34.0 -> 0.00 mm
- net button2: track 32.1 -> 0.00 mm
- net button1: track 31.9 -> 0.00 mm
- net GND: track 67.6 -> 36.0 mm, vias 0 -> 2
- net Net-(R1-Pad1): track 30.0 -> 0.00 mm
- net pH+: track 28.2 -> 0.00 mm
- net pH-: track 27.4 -> 0.00 mm
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Other:
- board text added: "3.3V"
- board text added: "GND"
- board text added: "ardHydroponic, ESP shield Design: Jon Sagebrand github.com/jonsag"
- board text removed: "ardHydroponic Design: Jon Sagebrand github.com/jonsag"

Commit message: pcb layout
Parts:
- added J1: LCD display, My_Headers:4-pin_I2C_LCD_header_larger, F.Cu at (185.4, 87.6)
- added J2: Buttons, My_Parts:6-pole_5-NO_switch_screw_terminal, F.Cu at (138.4, 90.8)
- added J3: MOSFETs, My_Parts:7-pole_6-MOSFET_screw_terminal, F.Cu at (176.7, 90.8)
- added R1: 4.7k, My_Misc:R_Axial_DIN0207_L6.3mm_D2.5mm_P10.16mm_Horizontal_larger_pads, F.Cu at (182.2, 104.1)
- added R2: 10k, My_Misc:R_Axial_DIN0207_L6.3mm_D2.5mm_P10.16mm_Horizontal_larger_pads, F.Cu at (134.0, 114.3)
- added R3: 10k, My_Misc:R_Axial_DIN0207_L6.3mm_D2.5mm_P10.16mm_Horizontal_larger_pads, F.Cu at (129.5, 114.3)
- added R4: 10k, My_Misc:R_Axial_DIN0207_L6.3mm_D2.5mm_P10.16mm_Horizontal_larger_pads, F.Cu at (125.1, 114.3)
- added R5: 10k, My_Misc:R_Axial_DIN0207_L6.3mm_D2.5mm_P10.16mm_Horizontal_larger_pads, F.Cu at (120.7, 114.3)
- added R6: 10k, My_Misc:R_Axial_DIN0207_L6.3mm_D2.5mm_P10.16mm_Horizontal_larger_pads, F.Cu at (116.2, 114.3)
- added U1: DS18B20, My_Parts:3-pole_DS18B20_screw_terminal, F.Cu at (154.9, 113.7)
- added U2: pH sensor, My_Headers:3-pin_DFRobot_Gravity_pH-sensor_header_large, F.Cu at (139.1, 106.7)
- added U3: TDS meter, My_Headers:3-pin_DFRobot_Gravity_TDS-meter_header_large, F.Cu at (146.1, 106.7)
- added U4: Power in, My_Parts:2-pole_power_in_screw_terminal, F.Cu at (104.8, 105.4)
- moved R8 54.2 mm to (177.8, 114.3), turned to 90 degrees
- moved R7 49.6 mm to (173.4, 104.1), turned to 270 degrees
- moved U10 20.4 mm to (163.8, 105.4), turned to 0 degrees
Connections:
- R7 pad 1: softTx -> Tx
- U10 pad 1: softRx -> Rx
- XA1 pad 100: +6V -> Net-(U4-Pad1)
- XA1 pad 25: softRx -> espReset
- XA1 pad 26: softTx -> Net-(XA1-Pad26)
- XA1 pad 45: Net-(XA1-Pad45) -> Rx
- XA1 pad 46: Net-(XA1-Pad46) -> Tx
- XA1 pad 64: espReset -> Net-(XA1-Pad30)
Routing:
- net +5V: track 0.00 -> 160.5 mm
- net GND: track 36.0 -> 136.0 mm, vias 2 -> 0
- net Net-(XA1-Pad30): track 0.00 -> 86.9 mm
- net Rx: track 0.00 -> 75.8 mm
- net softRx: track 51.2 -> 0.00 mm
- net Net-(U4-Pad1): track 0.00 -> 49.5 mm
- net Net-(R1-Pad1): track 0.00 -> 48.5 mm
- net button5: track 0.00 -> 43.8 mm
- net button4: track 0.00 -> 41.1 mm
- net button3: track 0.00 -> 38.5 mm
- net button2: track 0.00 -> 36.6 mm
- net button1: track 0.00 -> 35.9 mm
- net Tx: track 0.00 -> 34.8 mm
- net Net-(R7-Pad2): track 35.1 -> 12.0 mm
- net pH+: track 0.00 -> 20.4 mm
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- removed copper zone on B.Cu, net (none)
- removed copper zone on F.Cu, net (none)
- removed copper zone on B.Cu, net GND
- removed copper zone on F.Cu, net GND
Other:
- board size 102.9 x 54.6 mm -> 101.6 x 53.3 mm
- board text added: "ardHydroponic-v1.0RC1 Design: Jon Sagebrand github.com/jonsag"
- board text removed: "3.3V"
- board text removed: "GND"
- board text removed: "ardHydroponic, ESP shield Design: Jon Sagebrand github.com/jonsag"

Commit message: schematics
Parts:
- added K1: KY-019_relay_module, My_Headers:3-pin_KY-019_Relay_header_larger_pads, F.Cu at (185.4, 94.0)
Connections:
- U10 pad 4: Net-(U10-Pad4) -> Relay
Routing:
- net +3V3: track 40.9 -> 94.0 mm
- net Net-(XA1-Pad30): track 86.9 -> 133.6 mm
- net GND: track 136.0 -> 180.3 mm
- net +5V: track 160.5 -> 122.8 mm
- net Relay: track 0.00 -> 34.5 mm
- net Rx: track 75.8 -> 44.5 mm, vias 0 -> 1
- net Net-(U4-Pad1): track 49.5 -> 61.7 mm, vias 0 -> 2
- net Net-(R1-Pad1): track 48.5 -> 54.8 mm
- net Tx: track 34.8 -> 33.5 mm
- net espReset: track 55.2 -> 53.9 mm
- net button4: track 41.1 -> 40.1 mm
- net button5: track 43.8 -> 42.8 mm
- net Net-(U2-Pad3): track 17.7 -> 18.2 mm
