File: KiCAD/ardHydroponic/ardHydroponic.kicad_pcb (KiCad board)
At the start: 2 copper layers, 101.6 x 53.3 mm, 19 parts, among them J1 LCD display, J2 Buttons, J3 MOSFETs, K1 KY-019_relay_module, U1 DS18B20, U10 ESP-01, U2 pH sensor, U3 TDS meter, U4 Power in

Commit message: kicad6
Other:
- net class Default removed

Commit message: kicad6
Parts:
- U10: footprint My_Arduino:ESP-01_large -> My_Arduino:ESP-01_w_pin_socket_large
- moved XA1 54.2 mm to (119.1, 73.7)
- moved U10 0.25 mm to (164.1, 105.4)
- moved JP1 0.18 mm to (122.4, 120.1)
Connections:
- U10 pad 1: Rx -> GND
- U10 pad 2: GND -> Rx
- U10 pad 3: +3V3 -> Relay
- U10 pad 4: Relay -> +3V3
- U10 pad 5: espReset -> unconnected-(U10-Pad5)
- U10 pad 6: Net-(U10-Pad6) -> espReset
- U10 pad 7: +3V3 -> Net-(R7-Pad2)
- U10 pad 8: Net-(R7-Pad2) -> +3V3
- XA1 pad 11: Net-(XA1-Pad11) -> unconnected-(XA1-Pad11)
- XA1 pad 12: Net-(XA1-Pad12) -> unconnected-(XA1-Pad12)
- XA1 pad 13: Net-(XA1-Pad13) -> unconnected-(XA1-Pad13)
- XA1 pad 19: Net-(XA1-Pad19) -> unconnected-(XA1-Pad19)
- XA1 pad 2: Net-(XA1-Pad2) -> unconnected-(XA1-Pad2)
- XA1 pad 20: Net-(XA1-Pad20) -> unconnected-(XA1-Pad20)
- XA1 pad 21: Net-(XA1-Pad21) -> unconnected-(XA1-Pad21)
- XA1 pad 22: Net-(XA1-Pad22) -> unconnected-(XA1-Pad22)
- XA1 pad 26: Net-(XA1-Pad26) -> unconnected-(XA1-Pad26)
- XA1 pad 3: Net-(XA1-Pad3) -> unconnected-(XA1-Pad3)
- XA1 pad 31: Net-(XA1-Pad31) -> unconnected-(XA1-Pad31)
- XA1 pad 32: Net-(XA1-Pad32) -> unconnected-(XA1-Pad32)
- XA1 pad 35: Net-(XA1-Pad35) -> unconnected-(XA1-Pad35)
- XA1 pad 36: Net-(XA1-Pad36) -> unconnected-(XA1-Pad36)
- XA1 pad 37: Net-(XA1-Pad37) -> unconnected-(XA1-Pad37)
- XA1 pad 38: Net-(XA1-Pad38) -> unconnected-(XA1-Pad38)
- XA1 pad 39: Net-(XA1-Pad39) -> unconnected-(XA1-Pad39)
- XA1 pad 40: Net-(XA1-Pad40) -> unconnected-(XA1-Pad40)
- XA1 pad 41: Net-(XA1-Pad41) -> unconnected-(XA1-Pad41)
- XA1 pad 42: Net-(XA1-Pad42) -> unconnected-(XA1-Pad42)
- XA1 pad 50: Net-(XA1-Pad50) -> unconnected-(XA1-Pad50)
- XA1 pad 51: Net-(XA1-Pad51) -> unconnected-(XA1-Pad51)
- XA1 pad 52: Net-(XA1-Pad52) -> unconnected-(XA1-Pad52)
- XA1 pad 53: Net-(XA1-Pad53) -> unconnected-(XA1-Pad53)
- XA1 pad 54: Net-(XA1-Pad54) -> unconnected-(XA1-Pad54)
- XA1 pad 55: Net-(XA1-Pad55) -> unconnected-(XA1-Pad55)
- XA1 pad 56: Net-(XA1-Pad56) -> unconnected-(XA1-Pad56)
- XA1 pad 57: Net-(XA1-Pad57) -> unconnected-(XA1-Pad57)
- XA1 pad 58: Net-(XA1-Pad58) -> unconnected-(XA1-Pad58)
- XA1 pad 59: Net-(XA1-Pad59) -> unconnected-(XA1-Pad59)
- XA1 pad 60: Net-(XA1-Pad60) -> unconnected-(XA1-Pad60)
- XA1 pad 61: Net-(XA1-Pad61) -> unconnected-(XA1-Pad61)
- XA1 pad 63: Net-(XA1-Pad63) -> unconnected-(XA1-Pad63)
- XA1 pad 70: Net-(XA1-Pad70) -> unconnected-(XA1-Pad70)
- XA1 pad 71: Net-(XA1-Pad71) -> unconnected-(XA1-Pad71)
- XA1 pad 72: Net-(XA1-Pad72) -> unconnected-(XA1-Pad72)
- XA1 pad 73: Net-(XA1-Pad73) -> unconnected-(XA1-Pad73)
- XA1 pad 74: Net-(XA1-Pad74) -> unconnected-(XA1-Pad74)
- XA1 pad 75: Net-(XA1-Pad75) -> unconnected-(XA1-Pad75)
- XA1 pad 76: Net-(XA1-Pad76) -> unconnected-(XA1-Pad76)
- XA1 pad 77: Net-(XA1-Pad77) -> unconnected-(XA1-Pad77)
- XA1 pad 78: Net-(XA1-Pad78) -> unconnected-(XA1-Pad78)
- XA1 pad 81: Net-(XA1-Pad81) -> unconnected-(XA1-Pad81)
- XA1 pad 82: Net-(XA1-Pad82) -> unconnected-(XA1-Pad82)
- XA1 pad 83: Net-(XA1-Pad83) -> unconnected-(XA1-Pad83)
- XA1 pad 84: Net-(XA1-Pad84) -> unconnected-(XA1-Pad84)
- XA1 pad 85: Net-(XA1-Pad85) -> unconnected-(XA1-Pad85)
- XA1 pad 86: Net-(XA1-Pad86) -> unconnected-(XA1-Pad86)
- XA1 pad 87: Net-(XA1-Pad87) -> unconnected-(XA1-Pad87)
- XA1 pad 88: Net-(XA1-Pad88) -> unconnected-(XA1-Pad88)
- XA1 pad 89: Net-(XA1-Pad89) -> unconnected-(XA1-Pad89)
- XA1 pad 90: Net-(XA1-Pad90) -> unconnected-(XA1-Pad90)
- XA1 pad 91: Net-(XA1-Pad91) -> unconnected-(XA1-Pad91)
- XA1 pad 92: Net-(XA1-Pad92) -> unconnected-(XA1-Pad92)
- XA1 pad 93: Net-(XA1-Pad93) -> unconnected-(XA1-Pad93)
- XA1 pad 94: Net-(XA1-Pad94) -> unconnected-(XA1-Pad94)
- XA1 pad 98: Net-(XA1-Pad98) -> unconnected-(XA1-Pad98)
- XA1 pad 99: Net-(XA1-Pad99) -> unconnected-(XA1-Pad99)
- XA1 pad IORF: Net-(XA1-PadIORF) -> unconnected-(XA1-PadIORF)
- XA1 pad SCL: Net-(XA1-PadSCL) -> unconnected-(XA1-PadSCL)
- XA1 pad SDA: Net-(XA1-PadSDA) -> unconnected-(XA1-PadSDA)
Routing:
- net Net-(R1-Pad1): track 48.5 -> 51.7 mm
- net GND: track 184.9 -> 187.9 mm
- net Net-(JP1-Pad2): track 137.2 -> 134.7 mm
- net espReset: track 57.2 -> 55.2 mm
- net Rx: track 51.7 -> 49.9 mm
- net Net-(U4-Pad1): track 73.4 -> 71.7 mm
- net +5V: track 136.1 -> 135.0 mm
- net Relay: track 23.3 -> 22.2 mm
- net button1: track 42.2 -> 41.3 mm
- net Net-(J1-Pad5): track 13.6 -> 12.7 mm
- net Net-(U2-Pad3): track 28.8 -> 28.1 mm
- net +3V3: track 40.7 -> 41.4 mm
- net button5: track 46.5 -> 45.8 mm
- net Net-(JP1-Pad1): track 13.4 -> 12.8 mm
- net button3: track 43.1 -> 42.5 mm

Commit message: new pcb
Parts:
- removed J3: MOSFETs, My_Parts:7-pole_6-MOSFET_screw_terminal
- added U5: pH+ pump, My_Headers:3-pin JST IRF520 MOSFET module, F.Cu at (169.8, 87.0)
- added U6: pH- pump, My_Headers:3-pin JST IRF520 MOSFET module, F.Cu at (161.5, 87.0)
- added U7: nutr A pump, My_Headers:3-pin JST IRF520 MOSFET module, F.Cu at (153.3, 87.0)
- added U8: nutr B pump, My_Headers:3-pin JST IRF520 MOSFET module, F.Cu at (144.9, 87.0)
- added U9: stirrer, My_Headers:3-pin JST IRF520 MOSFET module, F.Cu at (136.7, 87.0)
- J1: value LCD display -> LCD 4x20; footprint My_Headers:4-pin_I2C_LCD_header_larger -> My_Headers:4-pin JST LCD
- J2: footprint My_Parts:6-pole_5-NO_switch_screw_terminal -> My_Headers:6-pin JST 5-buttons
- K1: footprint My_Headers:3-pin_KY-019_Relay_header_larger_pads -> My_Headers:3-pin JST KY-019 relay
- U1: footprint My_Parts:3-pole_DS18B20_screw_terminal -> My_Headers:3-pin JST DS18B20
- U2: footprint My_Headers:3-pin_DFRobot_Gravity_pH-sensor_header_large -> My_Headers:3-pin JST pH Sensor
- U3: footprint My_Headers:3-pin_DFRobot_Gravity_TDS-meter_header_large -> My_Headers:3-pin JST TDS Meter
- moved K1 40.6 mm to (144.1, 106.0), turned to -90 degrees
- moved U2 10.8 mm to (127.7, 96.6)
- moved U3 9.58 mm to (127.7, 108.7)
- moved J2 9.25 mm to (129.5, 88.3), turned to 180 degrees
- moved R2 8.25 mm to (121.3, 106.7)
- moved R3 8.25 mm to (116.8, 106.7)
- moved R4 8.25 mm to (112.4, 106.7)
- moved R5 8.25 mm to (108.0, 106.7)
- moved R6 8.25 mm to (103.5, 106.7)
- moved J1 7.96 mm to (177.2, 92.8), turned to 0 degrees
- moved U4 5.73 mm to (110.6, 77.0), turned to -90 degrees
Connections:
- J1 pad 3: GND -> Net-(XA1-Pad44)
- XA1 pad 43: Net-(J1-Pad7) -> Net-(XA1-Pad43)
- XA1 pad 44: Net-(J1-Pad5) -> Net-(XA1-Pad44)
Routing:
- net espReset: track 55.2 -> 121.3 mm
- net Net-(JP1-Pad2): track 134.7 -> 76.4 mm
- net GND: track 187.9 -> 230.5 mm
- net Net-(XA1-Pad43): track 0.00 -> 20.7 mm
- net Net-(XA1-Pad44): track 0.00 -> 19.6 mm
- net Net-(U3-Pad3): track 21.7 -> 35.3 mm, vias 0 -> 1
- net Net-(J1-Pad5): track 12.7 -> 0.00 mm
- net Relay: track 22.2 -> 33.3 mm
- net +5V: track 135.0 -> 145.6 mm, vias 0 -> 1
- net Net-(J1-Pad7): track 10.1 -> 0.00 mm
- net Rx: track 49.9 -> 42.6 mm, vias 2 -> 0
- net Net-(U2-Pad3): track 28.1 -> 33.1 mm, vias 1 -> 0
- net Net-(U4-Pad1): track 71.7 -> 67.8 mm, vias 1 -> 0
- net button1: track 41.3 -> 37.4 mm
- net button4: track 43.8 -> 40.1 mm
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- added copper zone on B.Cu, net (none)
- added copper zone on F.Cu, net (none)
- added copper zone on B.Cu, net GND
- added copper zone on F.Cu, net GND
Other:
- board text added: "1"
- board text added: "2"
- board text added: "3"
- board text added: "4"
- board text added: "5"
- board text added: "GND"
- board text added: "LCD"
- board text added: "Relay"
- board text added: "SIG"
- board text added: "Stirrer"
- board text added: "TDS- meter"
- board text added: "Temp sensor"
- board text added: "VCC"
- board text added: "ardHydroponic Design: Jon Sagebrand github.com/jonsag"
- board text added: "nutr A pump"
- board text added: "nutr B pump"
- board text added: "pH+ pump"
- board text added: "pH- meter"
- board text added: "pH- pump"
- board text removed: "Open to flash"
- board text removed: "ardHydroponic-v1.0RC1 Design: Jon Sagebrand github.com/jonsag"

Commit message: kicad
Other:
- board text added: "${TITLE}-${REVISION} Design: Jon Sagebrand github.com/jonsag"
- board text removed: "ardHydroponic Design: Jon Sagebrand github.com/jonsag"
Changed lines of the file:
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@@
   )
   (paper "A4")
+  (title_block
+    (title "ardHydroponic")
+    (date "2022-09-10")
+    (rev "0.2")
+  )
   (layers
     (0 "F.Cu" signal)
@@
     (effects (font (size 1 1) (thickness 0.15)))
   )
-  (gr_text "ardHydroponic\nDesign: Jon Sagebrand\ngithub.com/jonsag" (at 102.235 114.3) (layer "F.SilkS")
+  (gr_text "${TITLE}-${REVISION}\nDesign: Jon Sagebrand\ngithub.com/jonsag" (at 102.235 114.3) (layer "F.SilkS")
     (effects (font (size 1 1) (thickness 0.15)) (justify left))
   )
