File: KiCAD/ardHydroponic/ardHydroponic.kicad_sch (KiCad schematic)
At the start: 29 parts

Commit message: kicad6
Parts:
- removed JP1: (no value), symbol Device:Jumper
- removed U10: (no value), symbol ardHydroponic-rescue:ESP-01-My_Arduino
- added JP1: Flash, My_Parts:Jumper_1x02_P2.54mm_large, symbol Jumper:Jumper_2_Open
- added U10: ESP-01, My_Arduino:ESP-01_w_pin_socket_large, symbol My_Arduino:ESP-01
- J1: value (none) -> LCD display; footprint (none) -> My_Headers:4-pin_I2C_LCD_header_larger
- J2: value (none) -> Buttons; footprint (none) -> My_Parts:6-pole_5-NO_switch_screw_terminal
- J3: value (none) -> MOSFETs; footprint (none) -> My_Parts:7-pole_6-MOSFET_screw_terminal
- K1: value (none) -> KY-019_relay_module; footprint (none) -> My_Headers:3-pin_KY-019_Relay_header_larger_pads
- R1: value (none) -> 4.7k; footprint (none) -> My_Misc:R_Axial_DIN0207_L6.3mm_D2.5mm_P10.16mm_Horizontal_larger_pads
- R2, R3, R4, R5, R6: value (none) -> 10k; footprint (none) -> My_Misc:R_Axial_DIN0207_L6.3mm_D2.5mm_P10.16mm_Horizontal_larger_pads
- R7: value (none) -> 1k; footprint (none) -> My_Misc:R_Axial_DIN0207_L6.3mm_D2.5mm_P10.16mm_Horizontal_larger_pads
- R8: value (none) -> 2.2k; footprint (none) -> My_Misc:R_Axial_DIN0207_L6.3mm_D2.5mm_P10.16mm_Horizontal_larger_pads
- SW1: value (none) -> button1
- SW2: value (none) -> button2
- SW3: value (none) -> button3
- SW4: value (none) -> button4
- SW5: value (none) -> button5
- U1: value (none) -> DS18B20; footprint (none) -> My_Parts:3-pole_DS18B20_screw_terminal
- U2: value (none) -> pH sensor; footprint (none) -> My_Headers:3-pin_DFRobot_Gravity_pH-sensor_header_large
- U3: value (none) -> TDS meter; footprint (none) -> My_Headers:3-pin_DFRobot_Gravity_TDS-meter_header_large
- U4: value (none) -> Power in; footprint (none) -> My_Parts:2-pole_power_in_screw_terminal
- U5: value (none) -> pH+ pump
- U6: value (none) -> pH- pump
- U7: value (none) -> nutr A pump
- U8: value (none) -> nutr B pump
- U9: value (none) -> stirrer
- XA1: value (none) -> Arduino_Mega2560; footprint (none) -> My_Arduino:Arduino_Mega2560_Shield__no_ICSP_no_mount-holes_large
Connections:
- net +3V3: now also U10.4 (CH_PD/CH_EN), U10.8 (VCC)
- net GND: now also U10.1 (GND)
- net Relay: now also U10.3 (GPIO2)
- net Rx: now also U10.2 (GPIO1/UOTxD)
- net espReset: now also U10.6 (Reset)
- net at XA1.30 (RESET): now also JP1.1 (A)
- net at XA1.64 (D14_TX3): now also JP1.2 (B)
- net at R7.2, R8.1: now also U10.7 (GPIO3/UORxD)

Commit message: new pcb
Parts:
- removed J3: MOSFETs, My_Parts:7-pole_6-MOSFET_screw_terminal, symbol Connector:Screw_Terminal_01x07
- J1: value LCD display -> LCD 4x20; footprint My_Headers:4-pin_I2C_LCD_header_larger -> My_Headers:4-pin JST LCD
- J2: footprint My_Parts:6-pole_5-NO_switch_screw_terminal -> My_Headers:6-pin JST 5-buttons
- K1: footprint My_Headers:3-pin_KY-019_Relay_header_larger_pads -> My_Headers:3-pin JST KY-019 relay
- U1: footprint My_Parts:3-pole_DS18B20_screw_terminal -> My_Headers:3-pin JST DS18B20
- U2: footprint My_Headers:3-pin_DFRobot_Gravity_pH-sensor_header_large -> My_Headers:3-pin JST pH Sensor
- U3: footprint My_Headers:3-pin_DFRobot_Gravity_TDS-meter_header_large -> My_Headers:3-pin JST TDS Meter
- U5, U6, U7, U8, U9: footprint (none) -> My_Headers:3-pin JST IRF520 MOSFET module
Connections:
- net GND: now also J1.2 (GND); no longer J1.3 (GND)
- net at XA1.43 (D21_SCL): now also J1.4 (SCL); no longer J1.7 (SCL)
- net at XA1.44 (D20_SDA): now also J1.3 (SDA); no longer J1.5 (SDA)

Commit message: kicad
Other:
- title: (none) -> ardHydroponic
Changed lines of the file:
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@@
 (kicad_sch (version 20211123) (generator eeschema)
   (paper "A4")
+  (title_block
+    (title "ardHydroponic")
+    (date "2022-09-10")
+    (rev "0.2")
+  )
   (junction (at 193.04 118.11) (diameter 0) (color 0 0 0 0)
   )
