File: KiCAD/espProgrammerBoard/espProgrammerBoard.kicad_pcb (KiCad board)
At the start: 2 copper layers, 47 x 28.6 mm, 11 parts, among them J1 FTDI, J2 External power, SW1 Reset, SW2 Flash, U1 ESP-01

Commit message: text on copper
Other:
- board text added: "3.3V"
- board text added: "GND"

Commit message: kicad6
Parts:
- U1: footprint My_Arduino:ESP-01_large -> My_Arduino:ESP-01_w_pin_socket_large
Connections:
- J1 pad 2: Net-(J1-Pad2) -> unconnected-(J1-Pad2)
- J1 pad 6: Net-(J1-Pad6) -> unconnected-(J1-Pad6)
Routing:
- net Net-(J1-Pad4): track 35.2 -> 0.00 mm
- net +3V3: track 140.3 -> 175.5 mm
Other:
- net class Default removed

Commit message: programmer board
Parts:
- moved U1 0.38 mm to (127.4, 64.8)
Connections:
- U1 pad 1: Net-(J1-Pad5) -> GND
- U1 pad 2: GND -> Net-(J1-Pad5)
- U1 pad 3: +3V3 -> Net-(R1-Pad1)
- U1 pad 4: Net-(R1-Pad1) -> +3V3
- U1 pad 5: Net-(R2-Pad1) -> Net-(R3-Pad1)
- U1 pad 6: Net-(R3-Pad1) -> Net-(R2-Pad1)
- U1 pad 7: +3V3 -> Net-(J1-Pad4)
- U1 pad 8: Net-(J1-Pad4) -> +3V3
Routing:
- net Net-(J1-Pad4): track 0.00 -> 35.2 mm
- net +3V3: track 175.5 -> 140.3 mm
