File: KiCAD/espProgrammerBoard/espProgrammerBoard.kicad_sch (KiCad schematic)
At the start: 11 parts

Commit message: programmer board
Parts:
- removed U1: (no value), My_Arduino:ESP-01_w_pin_socket_large, symbol espProgrammerBoard-rescue:ESP-01-My_Arduino
- added U1: ESP-01, My_Arduino:ESP-01_w_pin_socket_large, symbol My_Arduino:ESP-01
- C1: value (none) -> 220u; footprint (none) -> My_Misc:CP_Radial_D6.3mm_P2.50mm_large
- C2: value (none) -> 100n; footprint (none) -> My_Misc:C_Disc_D3.0mm_W1.6mm_P2.50mm_larg
- J1: value (none) -> FTDI; footprint (none) -> My_Headers:6-pin_FTDI_header_large
- J2: value (none) -> External power; footprint (none) -> My_Headers:2-pin_power_input_header_larger_pads
- JP1: value (none) -> Power from FTDI; footprint (none) -> My_Parts:Jumper_1x02_P2.54mm_large
- R1, R2, R3: value (none) -> 10k; footprint (none) -> My_Misc:R_Axial_DIN0207_L6.3mm_D2.5mm_P10.16mm_Horizontal_larger_pads
- SW1: value (none) -> Reset; footprint (none) -> My_Misc:SW_PUSH_6mm_large
- SW2: value (none) -> Flash; footprint (none) -> My_Misc:SW_PUSH_6mm_large
Connections:
- net +3V3: now also U1.4 (CH_PD/CH_EN), U1.8 (VCC)
- net GND: now also U1.1 (GND)
- net at J1.4 (Tx): now also U1.7 (GPIO3/UORxD)
- net at J1.5 (Rx): now also U1.2 (GPIO1/UOTxD)
- net at R1.1: now also U1.3 (GPIO2)
- net at R2.1, SW1.1: now also U1.6 (Reset)
- net at R3.1, SW2.1: now also U1.5 (GPIO0/SPI_CS2)
Other:
- moved on the sheet: SW1, SW2
